File: dish_washwer_hardware/src/Steel_form_Dish_washer/_autosave-Steel_form_Dish_washer.kicad_pcb (KiCad board)
At the start: 2 copper layers, 230 x 287 mm, 152 parts, among them J1 RTD_TANK_SENSOR, J10 DRAIN PUMP CONNECTOR, J11 WASH PUMP CONNECTOR, J12 BOILER HEATER CONNECTOR, J13 TANK HEATER, J14 peristaltic_pump_2, J15 peristaltic_pump_1, J16 SCREEN CONNECTOR, J17 Conn_02x07_Odd_Even, J18 Conn_02x07_Odd_Even, J19 Pressure Switch 1, J2 RTD_BOILER_SENSOR, J20 Pressure Switch 2, J3 AC_PWR_IN, J4 MAG_DOOR_SENSOR, J5 Conn_02x03_Odd_Even, J6 Conn_01x04_Male, J7 Water sensor connector, J8 Conn_01x10_Male, J9 SOLENOID CONNECTOR, K1 9-1440003-0, K2 9-1440003-0, K3 9-1440003-0, K4 9-1440003-0, Q1 DMP6023LE-13, Q3 WST2N7002K, Q4 WST2N7002K, Q5 WST2N7002K, SW1 SW_Push, U1 ATmega2560-16AU, U10 MOC3021, U11 MOC3021, U12 MOC3021, U13 EL817, U15 TXS0108EPW, U16 EAST1616RGBA8, U17 EAST1616RGBA8, U18 MPR121QR2, U2 LM1117-3.3, U3 MAX31865ATP+T, U4 MAX31865ATP+T, U7 MOC3021, U8 MOC3021, U9 MOC3021, Y1 C3E-16.000-12-1010-M

Commit message: updated firmware
Connections:
- U1 pad 56: unconnected-(U1-Pad56) -> /WATER_LVL_LOW
- U1 pad 57: unconnected-(U1-Pad57) -> /WATER_LVL_HIGH
- U1 pad 88: /WATER_LVL_HIGH -> unconnected-(U1-Pad88)
- U1 pad 89: /WATER_LVL_LOW -> unconnected-(U1-Pad89)
Routing:
- net /WATER_LVL_HIGH: track 196.3 -> 182.5 mm
- net /WATER_LVL_LOW: track 186.3 -> 174.1 mm
- net /mcu_SCL: track 97.0 -> 97.5 mm
