File: dish_washwer_hardware/src/Steel_form_Dish_washer/AC_ACTUATORS.kicad_sch (KiCad schematic)
At the start: 65 parts, among them J10 DRAIN PUMP CONNECTOR, J11 WASH PUMP CONNECTOR, J12 BOILER HEATER CONNECTOR, J13 TANK HEATER, J14 peristaltic_pump_2, J15 peristaltic_pump_1, J19 Pressure Switch 1, J20 Pressure Switch 2, J7 Water sensor connector, J9 SOLENOID CONNECTOR, K1 9-1440003-0, K2 9-1440003-0, K3 9-1440003-0, K4 9-1440003-0, Q3 WST2N7002K, Q4 WST2N7002K, Q5 WST2N7002K, U10 MOC3021, U11 MOC3021, U12 MOC3021, U7 MOC3021, U8 MOC3021, U9 MOC3021

Commit message: updated firmware
Parts:
- gave numbers to parts that had none: 7
Changed lines of the file:
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@@
   (symbol (lib_id "Device:R_US") (at 63.754 211.709 180) (unit 1)
     (in_bom yes) (on_board yes)
-    (property "Reference" "R?" (id 0) (at 61.849 210.312 90)
+    (property "Reference" "R43" (id 0) (at 61.849 210.312 90)
       (effects (font (size 1.27 1.27)) (justify left))
     )
@@
   (symbol (lib_id "Device:R_US") (at 57.404 211.582 180) (unit 1)
     (in_bom yes) (on_board yes)
-    (property "Reference" "R?" (id 0) (at 55.499 210.185 90)
+    (property "Reference" "R42" (id 0) (at 55.499 210.185 90)
       (effects (font (size 1.27 1.27)) (justify left))
     )
@@
   (symbol (lib_id "power:+5V") (at 71.628 205.867 0) (unit 1)
     (in_bom yes) (on_board yes)
-    (property "Reference" "#PWR?" (id 0) (at 71.628 209.677 0)
+    (property "Reference" "#PWR036" (id 0) (at 71.628 209.677 0)
       (effects (font (size 1.27 1.27)) hide)
     )
@@
   (symbol (lib_id "Device:Q_PMOS_GDS") (at 302.514 203.2 0) (mirror x) (unit 1)
     (in_bom yes) (on_board yes) (fields_autoplaced)
-    (property "Reference" "Q?" (id 0) (at 308.61 201.9299 0)
+    (property "Reference" "Q1" (id 0) (at 308.61 201.9299 0)
       (effects (font (size 1.27 1.27)) (justify left))
     )
@@
   (symbol (lib_id "Device:R_US") (at 80.01 225.044 90) (unit 1)
     (in_bom yes) (on_board yes)
-    (property "Reference" "R?" (id 0) (at 77.343 224.028 90)
+    (property "Reference" "R46" (id 0) (at 77.343 224.028 90)
       (effects (font (size 1.27 1.27)) (justify left))
     )
@@
   (symbol (lib_id "power:+5V") (at 63.754 206.248 0) (unit 1)
     (in_bom yes) (on_board yes)
-    (property "Reference" "#PWR?" (id 0) (at 63.754 210.058 0)
+    (property "Reference" "#PWR035" (id 0) (at 63.754 210.058 0)
       (effects (font (size 1.27 1.27)) hide)
     )
@@
   (symbol (lib_id "Device:R_US") (at 80.391 222.504 90) (unit 1)
     (in_bom yes) (on_board yes)
-    (property "Reference" "R?" (id 0) (at 77.724 221.488 90)
+    (property "Reference" "R47" (id 0) (at 77.724 221.488 90)
       (effects (font (size 1.27 1.27)) (justify left))
     )
@@
   (symbol (lib_id "Device:R_US") (at 71.628 211.328 180) (unit 1)
     (in_bom yes) (on_board yes)
-    (property "Reference" "R?" (id 0) (at 69.723 209.931 90)
+    (property "Reference" "R44" (id 0) (at 69.723 209.931 90)
       (effects (font (size 1.27 1.27)) (justify left))
     )
@@
   (symbol (lib_id "Device:R_US") (at 79.502 227.584 90) (unit 1)
     (in_bom yes) (on_board yes)
-    (property "Reference" "R?" (id 0) (at 76.835 226.568 90)
-      (effects (font (size 1.27 1.27)) (justify left))
-    )
+    (property "Reference" "R45" (id 0) (at 76.835 226.568 90)
+      (effects (font (size 1.27 1.27)) (justify left))
+    )

Commit message: timing interrupt + pid
Parts:
- removed D5, D6: Q_TRIAC_A1A2G, Package_TO_SOT_THT:TO-220-3_Vertical, symbol Device:Q_TRIAC_A1A2G
- removed U11, U12: MOC3021, digikey-footprints:DIP-6_W7.62mm, symbol dk_Optoisolators-Triac-SCR-Output:MOC3021
- added K5, K6: 9-1440003-0, greencharge-footprints:TE_9-1440003-0, symbol 9-1440003-0:9-1440003-0
- added Q2, Q6: WST2N7002K, Package_TO_SOT_SMD:SOT-23, symbol Device:Q_NMOS_GDS
- R32, R33: value 200R -> 1K
Connections:
- net +5V: now also K5.1, K6.1
- net GND: now also R34.2, R35.2, Q2.3 (S), Q6.3 (S)
- net L1: now also K3.4; no longer K3.3
- net L3: now also K1.4, K2.4, K4.4, K5.4, K6.4; no longer K1.3, K2.3, K4.3, R34.1, R35.1
- net peristaltic_pump_1: now also R32.1; no longer R33.2
- net peristaltic_pump_2: now also R33.1; no longer R32.2
- net at RV11.1: now also J15.2 (Pin_2), K5.5; no longer J14.2 (Pin_2)
- net at RV12.1: now also J14.2 (Pin_2), K6.5; no longer J15.2 (Pin_2)
- new net: Q2.1 (G), R32.2, R34.1
- new net: K5.2, Q2.2 (D)
- new net: Q6.1 (G), R33.2, R35.1
- new net: K6.2, Q6.2 (D)
- no-connect marks 11 -> 10
Other:
- note added: "DRAIN PUMP PROBE CONTROLLED"
- moved on the sheet: D2, J13, J14, J15, K4, Q1, R16, R17, R27, R29, RV7, U8
