File: dish_washwer_hardware/src/AC_ACTUATORS.kicad_sch (KiCad schematic)
At the start: 65 parts, among them J10 SOLENOID CONNECTOR, J11 DRAIN PUMP CONNECTOR, J12 BOILER HEATER CONNECTOR, J13 Pressure Switch 1, J14 Pressure Switch 2, J15 peristaltic_pump_2, J16 peristaltic_pump_1, J17 TANK HEATER, J8 Water sensor connector, J9 WASH PUMP CONNECTOR, K1 9-1440003-0, K2 9-1440003-0, K3 9-1440003-0, K4 9-1440003-0, K5 9-1440003-0, K6 9-1440003-0, Q1 WST2N7002K, Q2 WST2N7002K, Q3 WST2N7002K, Q4 DMP6023L3-13, Q5 WST2N7002K, Q6 WST2N7002K, U11 MOC3021, U6 MOC3021, U7 MOC3021, U8 MOC3021

Commit message: cheaper version layout
Parts:
- removed J8: Water sensor connector, TerminalBlock_Phoenix:TerminalBlock_Phoenix_MKDS-1,5-4_1x04_P5.00mm_Horizontal, symbol Connector:Conn_01x04_Male
- removed Q1, Q2, Q3, Q5, Q6: WST2N7002K, Package_TO_SOT_SMD:SOT-23, symbol Device:Q_NMOS_GDS
- removed Q4: DMP6023L3-13, Package_TO_SOT_SMD:SOT-223-3_TabPin2, symbol Device:Q_PMOS_GDS
- added J8: Conn_01x03_Male, TerminalBlock_Phoenix:TerminalBlock_Phoenix_MKDS-1,5-3-5.08_1x03_P5.08mm_Horizontal, symbol Connector:Conn_01x03_Male
- added Q1, Q2, Q3, Q5, Q6: mmbt3904, Package_TO_SOT_SMD:SOT-23, symbol Device:Q_NPN_BEC
- added Q4: AP2301, Package_TO_SOT_SMD:SOT-23, symbol Device:Q_PMOS_GSD
- D4, D5, D6: MPN BTA30-600CW3G -> MAC223A6,127
- D7: renamed from D9; MPN BTA30-600CW3G -> MAC223A6,127
- J12: footprint greencharge-footprints:barrier_terminal_6PCV_04_006 -> greencharge-footprints:KF8500-4PIN
- J17: footprint greencharge-footprints:6PCV02006 -> greencharge-footprints:KF8500-2PIN
- K1, K2, K3, K4, K5, K6: value 9-1440003-0 -> SRA-05VDC-CL; footprint greencharge-footprints:TE_9-1440003-0 -> greencharge-footprints:SRA-05VDC-CL; Comment 9-1440003-0 -> SRA-05VDC-CL
- R20: renamed from R15; value 1K -> 800R
- R21: renamed from R16; value 1K -> 800R
- R22: renamed from R17; value 1K -> 800R
- R40: renamed from R48; value 1K -> 800R
- R41: renamed from R49; value 1K -> 800R
- RV10, RV11, RV12, RV4, RV5, RV6: value VDR-14D181K -> CNR-10D511KBTSA; footprint Varistor:RV_Disc_D16.5mm_W6.7mm_P7.5mm -> Varistor:RV_Disc_D15.5mm_W5.9mm_P7.5mm; MPN VDR-14D181K -> CNR-10D511KBTSA
- RV7, RV8, RV9: footprint Varistor:RV_Disc_D16.5mm_W6.7mm_P7.5mm -> Varistor:RV_Disc_D15.5mm_W5.9mm_P7.5mm
- renumbered J16 to J15, J15 to J16, R18 to R23, R19 to R24, R20 to R25, R30 to R26, R32 to R27, R33 to R28, R45 to R29, R46 to R30, R47 to R31, R21 to R32, R22 to R33, R23 to R34, R24 to R35, R25 to R36, R26 to R37, R27 to R38, R28 to R39, R50 to R42, R51 to R43, R31 to R44, R34 to R45, U6 to U5, U7 to U6, U8 to U7, U11 to U8
Connections:
- net +5V: now also Q4.2 (S)
- net E2: now also J8.1 (Pin_1)
- net E3: now also J8.2 (Pin_2)
- net GND: now also Q1.2 (E), Q2.2 (E), Q3.2 (E), Q5.2 (E), Q6.2 (E)
- net at K3.2: now also Q3.3 (C)
- net at R22.2, R25.1: now also Q3.1 (B)
- net at R21.2, R24.1: now also Q2.1 (B)
- net at K2.2: now also Q2.3 (C)
- net at K1.2: now also Q1.3 (C)
- net at R20.2, R23.1: now also Q1.1 (B)
- net at R28.2, R31.1: now also J8.3 (Pin_3)
- net at R38.2, R39.1: now also Q4.1 (G)
- net at K4.1: now also Q4.3 (D)
- net at R40.2, R42.1: now also Q5.1 (B)
- net at K5.2: now also Q5.3 (C)
- net at R41.2, R43.1: now also Q6.1 (B)
- net at K6.2: now also Q6.3 (C)
- no-connect marks 11 -> 10

Commit message: scare 1
Parts:
- added D10, D11, D12, D4, D5, D6: B5819WS, Diode_SMD:D_SOD-323, symbol Device:D_Schottky
- renumbered D7 to D13, D4 to D7, D5 to D8, D6 to D9
Connections:
- net +5V: now also D11.1 (K), D12.1 (K), D4.1 (K), D5.1 (K), D6.1 (K)
- net GND: now also D10.2 (A)
- net at K3.2, Q3.3 (C): now also D6.2 (A)
- net at K2.2, Q2.3 (C): now also D5.2 (A)
- net at K1.2, Q1.3 (C): now also D4.2 (A)
- net at K6.2, Q6.3 (C): now also D12.2 (A)
- net at K4.1, Q4.3 (D): now also D10.1 (K)
- net at K5.2, Q5.3 (C): now also D11.2 (A)
