File: dish_washwer_hardware/src/Steel_form_Dish_washer.kicad_sch (KiCad schematic)
At the start: 63 parts, among them J1 RTD_TANK_SENSOR, J2 RTD_BOILER_SENSOR, J3 AC_PWR_IN, J4 MAG_DOOR_SENSOR, J5 Conn_02x07_Odd_Even, J6 Conn_02x03_Odd_Even, J7 Conn_01x04_Male, SW1 SW_Push, U1 MAX31865ATP+T, U2 MAX31865ATP+T, U3 LM1117-3.3, U4 ATmega2560-16AU, U5 EL817, Y1 C3E-16.000-12-1010-M

Commit message: cheaper version layout
Parts:
- removed C1, C10, C2, C5, C6, C9: 100nF, Capacitor_SMD:C_0402_1005Metric, symbol Device:C_Small
- removed J1: RTD_TANK_SENSOR, Connector_JST:JST_EH_S3B-EH_1x03_P2.50mm_Horizontal, symbol Connector:Conn_01x03_Male
- removed J2: RTD_BOILER_SENSOR, Connector_JST:JST_EH_S3B-EH_1x03_P2.50mm_Horizontal, symbol Connector:Conn_01x03_Male
- removed J3: AC_PWR_IN, greencharge-footprints:387207505, symbol Connector:Conn_01x05_Male
- removed PS1: HLK-5M05, greencharge-footprints:CONV_HLK-5M05, symbol HLK-5M05:HLK-5M05
- removed U1, U2: MAX31865ATP+T, greencharge-footprints:QFN65P500X500X80-21N, symbol MAX31865ATP_T:MAX31865ATP+T
- added J1: RTD_BOILER_SENSOR, Connector_JST:JST_EH_S2B-EH_1x02_P2.50mm_Horizontal, symbol Connector:Conn_01x02_Male
- added J2: AC_PWR_IN, greencharge-footprints:KF8500-4PIN, symbol Connector:Conn_01x04_Male
- added J3: RTD_TANK_SENSOR, Connector_JST:JST_EH_S2B-EH_1x02_P2.50mm_Horizontal, symbol Connector:Conn_01x02_Male
- added PS1: HLK-PM01, Converter_ACDC:Converter_ACDC_HiLink_HLK-PMxx, symbol Converter_ACDC:HLK-PM01
- added R3, R4, R6: 10K, Resistor_SMD:R_0402_1005Metric, symbol Device:R_US
- added R5: 1K, Resistor_SMD:R_0402_1005Metric, symbol Device:R_US
- added U1: LM358, Package_SO:SO-8_3.9x4.9mm_P1.27mm, symbol Amplifier_Operational:LM358
- R1: value 4300 R_0.1% -> 10K
- R2: value 4300 R_0.1% -> 1K
- RV1, RV2, RV3: value VDR-14D181K -> CNR-10D511KBTSA; footprint Varistor:RV_Disc_D16.5mm_W6.7mm_P7.5mm -> Varistor:RV_Disc_D15.5mm_W5.9mm_P7.5mm; MPN VDR-14D181K -> CNR-10D511KBTSA
- U2: renamed from U3; value LM1117-3.3 -> AMS1117-3.3
- Y1: value C3E-16.000-12-1010-M -> 16MHz; MPN (none) -> S3216000091060
- renumbered C3 to C1, C16 to C10, C17 to C11, C18 to C12, C19 to C13, C20 to C14, C21 to C15, C22 to C16, C4 to C2, C7 to C3, C8 to C4, C11 to C5, C12 to C6, C13 to C7, C14 to C8, C15 to C9, R5 to R10, R6 to R11, R7 to R12, R8 to R13, R9 to R14, R10 to R15, R11 to R16, R12 to R17, R13 to R18, R14 to R19, R3 to R7, R29 to R8, R4 to R9, U4 to U3, U5 to U4
Connections:
- net BIAS is gone; now on net +5V: R1.1
- net BIAS1 is gone; now on an unnamed net: R2.1
- net +5V: now also PS1.4 (+Vout), R3.1, R4.1, R6.1, U1.8 (V+)
- net GND: now also R2.2, J1.2 (Pin_2), J3.2 (Pin_2), PS1.3 (-Vout), R5.2, U1.4 (V-)
- net L1: now also J2.1 (Pin_1)
- net L2: now also J2.2 (Pin_2)
- net L3: now also J2.3 (Pin_3), PS1.1 (AC/L)
- net NEUTRAL: now also J2.4 (Pin_4), PS1.2 (AC/N)
- net BOILER_RTD: now reaches U3.88 (PK1)
- net BOILER_RTD: now also U1.7
- net TANK_RTD: now reaches U3.89 (PK0)
- net TANK_RTD: now also U1.1
- net at R1.2: now also U1.6 (-)
- net RTD_SCLK renamed SCK
- net RTD_~{CS_1}: no longer names the net of U3.19 (PB0)
- net RTD_~{CS}: no longer names the net of U3.24 (PB5)
- net RTD_~{DRDY}: no longer names the net of U3.23 (PB4)
- new net: J1.1 (Pin_1), R3.2, U1.5 (+)
- new net: R4.2, R5.1, U1.2 (-)
- new net: J3.1 (Pin_1), R6.2, U1.3 (+)
- no-connect marks 50 -> 51
Other:
- note added: "PT1000 2-WIRE"
- note added: "RTD SENSOR INTERFACE (PT1000 2WIRER )"
- note removed: "3 WIRE SENSOR CONNECTION"
- note removed: "PT1000 3-WIRE"
- note removed: "RTD SENSOR INTERFACE(PT1000)"
- note removed: "Rref= 430R which is connected to the bias pin"

Commit message: scare 1
Connections:
- net +3V3: no longer R14.1
- net +5V: now also R14.1
- net RTD_~{DRDY_1}: no longer names the net of U3.25 (PB6)
- no-connect marks 51 -> 52
Changed lines of the file:
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@@
   (no_connect (at 231.14 117.602))
   (no_connect (at 247.65 122.682))
+  (no_connect (at 242.57 76.962))
   (no_connect (at 190.5 71.882))
   (no_connect (at 231.14 125.222))
@@
     (effects (font (size 0.9906 0.9906)) (justify left bottom))
   )
-  (label "RTD_~{DRDY_1}" (at 242.57 76.962 0)
-    (effects (font (size 0.9906 0.9906)) (justify left bottom))
-  )
   (label "MOSI" (at 372.237 163.576 0)
     (effects (font (size 0.9906 0.9906)) (justify left bottom))
@@
     (pin "1")
   )
+  (symbol (lib_id "power:+5V") (at 264.287 156.972 0) (unit 1)
+    (in_bom yes) (on_board yes)
+    (property "Reference" "#PWR?" (id 0) (at 264.287 160.782 0)
+      (effects (font (size 1.27 1.27)) hide)
+    )
+    (property "Value" "+5V" (id 1) (at 263.525 152.654 0))
+    (property "Footprint" "" (id 2) (at 264.287 156.972 0)
+      (effects (font (size 1.27 1.27)) hide)
+    )
+    (property "Datasheet" "" (id 3) (at 264.287 156.972 0)
+      (effects (font (size 1.27 1.27)) hide)
+    )
+    (pin "1")
+  )
   (symbol (lib_id "power:GND") (at 256.921 46.228 0) (unit 1)
     (in_bom yes) (on_board yes)
@@
     (pin "1")
   )
-  (symbol (lib_id "power:+3.3V") (at 264.287 156.972 0) (unit 1)
-    (in_bom yes) (on_board yes)
-    (property "Reference" "#PWR031" (id 0) (at 264.287 160.782 0)
-      (effects (font (size 1.27 1.27)) hide)
-    )
-    (property "Value" "+3.3V" (id 1) (at 264.668 152.5778 0))
-    (property "Footprint" "" (id 2) (at 264.287 156.972 0)
-      (effects (font (size 1.27 1.27)) hide)
-    )
-    (property "Datasheet" "" (id 3) (at 264.287 156.972 0)
-      (effects (font (size 1.27 1.27)) hide)
-    )
-    (pin "1")
-  )
   (symbol (lib_id "power:GND") (at 369.189 90.932 90) (unit 1)
     (in_bom yes) (on_board yes)
@@
       (reference "#PWR030") (unit 1) (value "+5V") (footprint "")
     )
-    (path "/b189f980-2467-4de3-b9eb-07f9e8037e23"
-      (reference "#PWR031") (unit 1) (value "+3.3V") (footprint "")
-    )
     (path "/00000000-0000-0000-0000-0000648067ef"
       (reference "#PWR032") (unit 1) (value "GND1") (footprint "")
@@
       (reference "#PWR096") (unit 1) (value "GND") (footprint "")
     )
+    (path "/8e9d6d7a-f63f-4508-aa8f-bb3a5ec903da"
+      (reference "#PWR?") (unit 1) (value "+5V") (footprint "")
+    )
     (path "/bec2222d-e897-45a4-9a97-9dfbdc08b2b2"
       (reference "BZ1") (unit 1) (value "PS1240P02BT") (footprint "digikey-footprints:Piezo_Transducer_THT_PS1240P02BT")
@@
       (reference "D3") (unit 1) (value "MB6S") (footprint "Package_TO_SOT_SMD:TO-269AA")
     )
+    (path "/00000000-0000-0000-0000-00006384df38/8c630a40-2342-4ebf-93fe-e61c5f19ef3f"
+      (reference "D4") (unit 1) (value "B5819WS") (footprint "Diode_SMD:D_SOD-323")
+    )
+    (path "/00000000-0000-0000-0000-00006384df38/27ca6772-3415-4903-b4b1-4699fbe0291d"
+      (reference "D5") (unit 1) (value "B5819WS") (footprint "Diode_SMD:D_SOD-323")
+    )
+    (path "/00000000-0000-0000-0000-00006384df38/5f018de3-1552-4135-a3eb-37a3706e4ab5"
+      (reference "D6") (unit 1) (value "B5819WS") (footprint "Diode_SMD:D_SOD-323")
+    )
     (path "/00000000-0000-0000-0000-00006384df38/00000000-0000-0000-0000-0000638c11ea"
-      (reference "D4") (unit 1) (value "Q_TRIAC_A1A2G") (footprint "Package_TO_SOT_THT:TO-220-3_Vertical")
+      (reference "D7") (unit 1) (value "Q_TRIAC_A1A2G") (footprint "Package_TO_SOT_THT:TO-220-3_Vertical")
     )
     (path "/00000000-0000-0000-0000-00006384df38/00000000-0000-0000-0000-0000638c11b3"
-      (reference "D5") (unit 1) (value "Q_TRIAC_A1A2G") (footprint "Package_TO_SOT_THT:TO-220-3_Vertical")
+      (reference "D8") (unit 1) (value "Q_TRIAC_A1A2G") (footprint "Package_TO_SOT_THT:TO-220-3_Vertical")
     )
     (path "/00000000-0000-0000-0000-00006384df38/00000000-0000-0000-0000-0000638c1221"
-      (reference "D6") (unit 1) (value "Q_TRIAC_A1A2G") (footprint "Package_TO_SOT_THT:TO-220-3_Vertical")
+      (reference "D9") (unit 1) (value "Q_TRIAC_A1A2G") (footprint "Package_TO_SOT_THT:TO-220-3_Vertical")
+    )
+    (path "/00000000-0000-0000-0000-00006384df38/49340243-2111-46bb-b34c-4b4e49f49d8b"
+      (reference "D10") (unit 1) (value "B5819WS") (footprint "Diode_SMD:D_SOD-323")
+    )
+    (path "/00000000-0000-0000-0000-00006384df38/ec72bdc3-8b93-4e8b-a59d-4599e176d60e"
+      (reference "D11") (unit 1) (value "B5819WS") (footprint "Diode_SMD:D_SOD-323")
+    )
+    (path "/00000000-0000-0000-0000-00006384df38/51b19f27-3541-4f08-9c1a-43541f27c269"
+      (reference "D12") (unit 1) (value "B5819WS") (footprint "Diode_SMD:D_SOD-323")
     )
     (path "/00000000-0000-0000-0000-00006384df38/00000000-0000-0000-0000-0000638c118d"
-      (reference "D7") (unit 1) (value "Q_TRIAC_A1A2G") (footprint "Package_TO_SOT_THT:TO-220-3_Vertical")
+      (reference "D13") (unit 1) (value "Q_TRIAC_A1A2G") (footprint "Package_TO_SOT_THT:TO-220-3_Vertical")
     )
     (path "/dab3b635-129e-4561-8546-e374aa73302a"
