File: dish_washwer_hardware/src/Steel_form_Dish_washer PART 1.kicad_pcb (KiCad board)
At the start: 4 copper layers, 185 x 95 mm, 128 parts, among them J1 RTD_TANK_SENSOR, J10 SOLENOID CONNECTOR, J11 DRAIN PUMP CONNECTOR, J12 BOILER HEATER CONNECTOR, J13 Pressure Switch 1, J14 Pressure Switch 2, J15 peristaltic_pump_2, J16 peristaltic_pump_1, J17 TANK HEATER, J2 RTD_BOILER_SENSOR, J3 AC_PWR_IN, J4 MAG_DOOR_SENSOR, J5 Conn_02x07_Odd_Even, J6 Conn_02x03_Odd_Even, J7 Conn_01x04_Male, J8 Water sensor connector, J9 WASH PUMP CONNECTOR, K1 9-1440003-0, K2 9-1440003-0, K3 9-1440003-0, K4 9-1440003-0, K5 9-1440003-0, K6 9-1440003-0, Q1 WST2N7002K, Q2 WST2N7002K, Q3 WST2N7002K, Q4 DMP6023L3-13, Q5 WST2N7002K, Q6 WST2N7002K, SW1 SW_Push, U1 MAX31865ATP+T, U11 MOC3021, U2 MAX31865ATP+T, U3 LM1117-3.3, U4 ATmega2560-16AU, U5 EL817, U6 MOC3021, U7 MOC3021, U8 MOC3021, Y1 C3E-16.000-12-1010-M

Commit message: complete layout and schematic
Parts:
- removed C17: 4.7nF, Capacitor_SMD:C_0402_1005Metric
- removed C18, C19, C20, C21, C22: 100nF, Capacitor_SMD:C_0402_1005Metric
- removed the D9 at (279.5, 92.3)
- removed R46, R47: 1M, Resistor_SMD:R_0402_1005Metric
- removed R48, R49: 1K, Resistor_SMD:R_0402_1005Metric
- removed R50, R51: 10K, Resistor_SMD:R_0402_1005Metric
- removed U11: MOC3021, digikey-footprints:DIP-6_W7.62mm
- added D10: B5819WS, Diode_SMD:D_SOD-323, F.Cu at (269.4, 148.8)
- added D11: B5819WS, Diode_SMD:D_SOD-323, F.Cu at (256.1, 89.5)
- added D12: B5819WS, Diode_SMD:D_SOD-323, F.Cu at (159.1, 75.5)
- added D13: Q_TRIAC_A1A2G, Package_TO_SOT_THT:TO-220-3_Vertical, F.Cu at (281.1, 79.6)
- added D4: B5819WS, Diode_SMD:D_SOD-323, F.Cu at (251.3, 104.0)
- added D5: B5819WS, Diode_SMD:D_SOD-323, F.Cu at (251.3, 118.5)
- added D6: B5819WS, Diode_SMD:D_SOD-323, F.Cu at (251.1, 136.3)
- added R35: 10K, Resistor_SMD:R_0402_1005Metric, F.Cu at (223.8, 82.8)
- added R36: 10K, Resistor_SMD:R_0402_1005Metric, F.Cu at (169.3, 81.7)
- added R37: 10K, Resistor_SMD:R_0402_1005Metric, F.Cu at (196.7, 82.8)
- added R38: 1K, Resistor_SMD:R_0402_1005Metric, F.Cu at (264.9, 146.3)
- added R39: 10K, Resistor_SMD:R_0402_1005Metric, F.Cu at (264.9, 151.1)
- added R40: 800R, Resistor_SMD:R_0402_1005Metric, F.Cu at (250.3, 91.5)
- added R41: 800R, Resistor_SMD:R_0402_1005Metric, F.Cu at (161.7, 75.0)
- added R42: 10K, Resistor_SMD:R_0402_1005Metric, F.Cu at (255.1, 91.5)
- added R43: 10K, Resistor_SMD:R_0402_1005Metric, F.Cu at (161.7, 70.3)
- added R44: 200R, Resistor_SMD:R_0402_1005Metric, F.Cu at (266.7, 81.1)
- C1: value 100nF -> 10uF
- C11: value 100nF -> 4.7nF
- C13: value 100u -> 100nF; footprint Capacitor_SMD:CP_Elec_5x5.4 -> Capacitor_SMD:C_0402_1005Metric
- C14, C15: value 22pF -> 100nF
- C2: value 100nF -> 1uF
- C3: value 10uF -> 100nF
- C4: value 1uF -> 100nF
- C7: value 100nF -> 100u; footprint Capacitor_SMD:C_0402_1005Metric -> Capacitor_SMD:CP_Elec_5x5.4
- C8, C9: value 100nF -> 22pF
- J1: value RTD_TANK_SENSOR -> RTD_BOILER_SENSOR; footprint Connector_JST:JST_EH_S3B-EH_1x03_P2.50mm_Horizontal -> Connector_JST:JST_EH_S2B-EH_1x02_P2.50mm_Horizontal
- J12: footprint greencharge-footprints:barrier_terminal_6PCV_04_006 -> greencharge-footprints:KF8500-4PIN
- J15: value peristaltic_pump_2 -> peristaltic_pump_1
- J16: value peristaltic_pump_1 -> peristaltic_pump_2
- J17: footprint greencharge-footprints:6PCV02006 -> greencharge-footprints:KF8500-2PIN
- J2: value RTD_BOILER_SENSOR -> AC_PWR_IN; footprint Connector_JST:JST_EH_S3B-EH_1x03_P2.50mm_Horizontal -> greencharge-footprints:KF8500-4PIN
- J3: value AC_PWR_IN -> RTD_TANK_SENSOR; footprint greencharge-footprints:387207505 -> Connector_JST:JST_EH_S2B-EH_1x02_P2.50mm_Horizontal
- J8: value Water sensor connector -> Conn_01x03_Male; footprint TerminalBlock_Phoenix:TerminalBlock_Phoenix_MKDS-1,5-4_1x04_P5.00mm_Horizontal -> TerminalBlock_Phoenix:TerminalBlock_Phoenix_MKDS-1,5-3-5.08_1x03_P5.08mm_Horizontal
- K1, K2, K3, K4, K5, K6: value 9-1440003-0 -> SRA-05VDC-CL; footprint greencharge-footprints:TE_9-1440003-0 -> greencharge-footprints:SRA-05VDC-CL
- PS1: value HLK-5M05 -> HLK-PM01; footprint greencharge-footprints:CONV_HLK-5M05 -> Converter_ACDC:Converter_ACDC_HiLink_HLK-PMxx
- Q1, Q2, Q3, Q5, Q6: value WST2N7002K -> mmbt3904
- Q4: value DMP6023L3-13 -> AP2301; footprint Package_TO_SOT_SMD:SOT-223-3_TabPin2 -> Package_TO_SOT_SMD:SOT-23
- R1: value 4300 R_0.1% -> 10K
- R10, R8: value 4.7k -> 10K
- R11: value 47K -> 500R; footprint Resistor_SMD:R_0805_2012Metric -> Resistor_SMD:R_0402_1005Metric
- R12: value 47K -> 4.7k; footprint Resistor_SMD:R_0805_2012Metric -> Resistor_SMD:R_0402_1005Metric
- R13: value 100R -> 4.7k; footprint Resistor_SMD:R_0603_1608Metric -> Resistor_SMD:R_0402_1005Metric
- R14, R15: value 1K -> 4.7k
- R16, R17: value 1K -> 47K; footprint Resistor_SMD:R_0402_1005Metric -> Resistor_SMD:R_0805_2012Metric
- R18: value 10K -> 100R; footprint Resistor_SMD:R_0402_1005Metric -> Resistor_SMD:R_0603_1608Metric
- R19, R26, R28, R5: value 10K -> 1K
- R2: value 4300 R_0.1% -> 1K
- R20: value 10K -> 800R
- R21, R22: value 200R -> 800R
- R23, R3: value 200R -> 10K
- R29: value 10K -> 1M
- R30: value 1K -> 1M
- R31: value 200R -> 1M
- R32, R33: value 1K -> 200R
- R34: value 10K -> 200R
- R4, R6: value 500R -> 10K
- R45: value 1M -> 10K
- R7: value 4.7k -> 200R
- R9: value 4.7k -> 500R
- RV1, RV10, RV11, RV12, RV2, RV3, RV4, RV5, RV6: value VDR-14D181K -> CNR-10D511KBTSA; footprint Varistor:RV_Disc_D16.5mm_W6.7mm_P7.5mm -> Varistor:RV_Disc_D15.5mm_W5.9mm_P7.5mm
- RV7, RV8, RV9: footprint Varistor:RV_Disc_D16.5mm_W6.7mm_P7.5mm -> Varistor:RV_Disc_D15.5mm_W5.9mm_P7.5mm
- U1: value MAX31865ATP+T -> LM358; footprint greencharge-footprints:QFN65P500X500X80-21N -> Package_SO:SO-8_3.9x4.9mm_P1.27mm
- U2: value MAX31865ATP+T -> AMS1117-3.3; footprint greencharge-footprints:QFN65P500X500X80-21N -> digikey-footprints:SOT-223
- U3: value LM1117-3.3 -> ATmega2560-16AU; footprint digikey-footprints:SOT-223 -> Package_QFP:TQFP-100_14x14mm_P0.5mm
- U4: value ATmega2560-16AU -> EL817; footprint Package_QFP:TQFP-100_14x14mm_P0.5mm -> Package_DIP:DIP-4_W7.62mm
- U5: value EL817 -> MOC3021; footprint Package_DIP:DIP-4_W7.62mm -> digikey-footprints:DIP-6_W7.62mm
- Y1: value C3E-16.000-12-1010-M -> 16MHz
- moved R31 126.5 mm to (172.5, 138.7), turned to 90 degrees
- moved R45 124.8 mm to (278.4, 81.0)
- moved RV11 110.9 mm to (139.6, 64.5)
- moved K6 103.5 mm to (155.1, 72.2), turned to -90 degrees
- moved Q6 101.3 mm to (160.7, 72.7)
- moved R17 98.8 mm to (152.8, 100.3)
- moved R34 96.8 mm to (185.2, 82.8), turned to 90 degrees
- moved R25 95.9 mm to (249.0, 135.1), turned to 0 degrees
- moved R16 93.9 mm to (152.7, 111.2)
- moved K5 92.9 mm to (262.5, 83.9), turned to -90 degrees
- moved J3 91.8 mm to (203.7, 145.6), turned to 180 degrees
- moved Q5 91.6 mm to (252.7, 90.5), turned to 90 degrees
- moved J2 91.1 mm to (133.4, 89.8), turned to -90 degrees
- moved R22 84.9 mm to (249.2, 130.2)
- moved U6 84.3 mm to (159.8, 81.2), turned to 0 degrees
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- renumbered D4 to D7, D5 to D8, D6 to D9
Connections:
- C1 pad 1: /RTD1_IN+ -> +5V
- C1 pad 2: /RTD1_IN- -> GND
- C10 pad 1: +3V3 -> Net-(C10-Pad1)
- C11 pad 1: +5V -> /RESET
- C14 pad 1: Net-(C14-Pad1) -> +5V
- C15 pad 1: Net-(C15-Pad1) -> +5V
- C16 pad 1: Net-(C16-Pad1) -> +5V
- C2 pad 1: /RTD2_IN+ -> +3V3
- C2 pad 2: /RTD2_IN- -> GND
- C4 pad 1: +3V3 -> +5V
- C5 pad 1: +3V3 -> +5V
- C6 pad 1: +3V3 -> +5V
- C8 pad 1: +5V -> Net-(C8-Pad1)
- C9 pad 1: +3V3 -> Net-(C9-Pad1)
- D7 pad 3: Net-(D4-Pad3) -> Net-(D7-Pad3)
- D8 pad 3: Net-(D5-Pad3) -> Net-(D8-Pad3)
- D9 pad 3: Net-(D6-Pad3) -> Net-(D9-Pad3)
- J1 pad 1: /RTD1_IN- -> Net-(J1-Pad1)
- J1 pad 2: /RTD1_IN+ -> GND
- J15 pad 1: NEUTRAL -> Net-(J15-Pad1)
- J15 pad 2: Net-(J15-Pad2) -> NEUTRAL
- J16 pad 1: Net-(J16-Pad1) -> NEUTRAL
- J16 pad 2: NEUTRAL -> Net-(J16-Pad2)
- J2 pad 1: /RTD2_IN- -> L1
- J2 pad 2: /RTD2_IN+ -> L2
- J2 pad 3: Net-(J2-Pad3) -> L3
- J3 pad 1: L1 -> Net-(J3-Pad1)
- J3 pad 2: L2 -> GND
- J6 pad 3: /RTD_SCLK -> /SCK
- J8 pad 1: unconnected-(J8-Pad1) -> /AC_ACTUATORS/E2
- J8 pad 2: /AC_ACTUATORS/E2 -> /AC_ACTUATORS/E3
- J8 pad 3: /AC_ACTUATORS/E3 -> Net-(J8-Pad3)
- K1 pad 2: Net-(K1-Pad2) -> Net-(D4-Pad2)
- K2 pad 2: Net-(K2-Pad2) -> Net-(D5-Pad2)
- K3 pad 2: Net-(K3-Pad2) -> Net-(D6-Pad2)
- K4 pad 1: Net-(K4-Pad1) -> Net-(D10-Pad1)
- K5 pad 2: Net-(K5-Pad2) -> Net-(D11-Pad2)
- K5 pad 5: Net-(J16-Pad1) -> Net-(J15-Pad1)
- K6 pad 2: Net-(K6-Pad2) -> Net-(D12-Pad2)
- K6 pad 5: Net-(J15-Pad2) -> Net-(J16-Pad2)
- Q1 pad 2: Net-(K1-Pad2) -> GND
- Q1 pad 3: GND -> Net-(D4-Pad2)
- Q2 pad 2: Net-(K2-Pad2) -> GND
- Q2 pad 3: GND -> Net-(D5-Pad2)
- Q3 pad 2: Net-(K3-Pad2) -> GND
- Q3 pad 3: GND -> Net-(D6-Pad2)
- Q4 pad 2: Net-(K4-Pad1) -> +5V
- Q4 pad 3: +5V -> Net-(D10-Pad1)
- Q5 pad 2: Net-(K5-Pad2) -> GND
- Q5 pad 3: GND -> Net-(D11-Pad2)
- Q6 pad 2: Net-(K6-Pad2) -> GND
- Q6 pad 3: GND -> Net-(D12-Pad2)
- R1 pad 1: /BIAS -> +5V
- R10 pad 2: /mcu_~{IRQ} -> /RESET
- R11 pad 1: L1 -> Net-(R11-Pad1)
- R11 pad 2: Net-(D3-Pad2) -> Net-(D2-Pad2)
- R12 pad 1: NEUTRAL -> +5V
- R12 pad 2: Net-(D3-Pad1) -> /mcu_SCL
- R13 pad 1: /SPEAKER -> +5V
- R13 pad 2: Net-(BZ1-Pad1) -> /mcu_SDA
- R14 pad 1: GND -> +5V
- R14 pad 2: /ZERO_CROSS_DETECT -> /mcu_SCREEN_RST
- R15 pad 1: /WASH_PUMP -> +5V
- R15 pad 2: Net-(Q1-Pad1) -> /mcu_~{IRQ}
- R16 pad 1: /DRAIN_PUMP -> L1
- R16 pad 2: Net-(Q2-Pad1) -> Net-(D3-Pad2)
- R17 pad 1: /SOLENOID -> NEUTRAL
- R17 pad 2: Net-(Q3-Pad1) -> Net-(D3-Pad1)
- R18 pad 1: Net-(Q1-Pad1) -> /SPEAKER
- R18 pad 2: GND -> Net-(BZ1-Pad1)
- R19 pad 1: Net-(Q2-Pad1) -> GND
- R19 pad 2: GND -> /ZERO_CROSS_DETECT
- R2 pad 1: /BIAS1 -> Net-(R1-Pad2)
- R2 pad 2: Net-(R2-Pad2) -> GND
- R20 pad 1: Net-(Q3-Pad1) -> /WASH_PUMP
- R20 pad 2: GND -> Net-(Q1-Pad1)
- R21 pad 1: Net-(R21-Pad1) -> /DRAIN_PUMP
- R21 pad 2: /L2_3phase_heater_pwm -> Net-(Q2-Pad1)
- R22 pad 1: Net-(R22-Pad1) -> /SOLENOID
- R22 pad 2: /L1_3phase_heater_pwm -> Net-(Q3-Pad1)
- R23 pad 1: Net-(R23-Pad1) -> Net-(Q1-Pad1)
- R23 pad 2: /L3_3phase_heater_pwm -> GND
- R24 pad 1: L2 -> Net-(Q2-Pad1)
- R24 pad 2: Net-(R24-Pad2) -> GND
- R25 pad 1: L1 -> Net-(Q3-Pad1)
- R25 pad 2: Net-(R25-Pad2) -> GND
- R26 pad 1: L3 -> +5V
- R26 pad 2: Net-(R26-Pad2) -> /AC_ACTUATORS/E2
- R27 pad 1: /AC_ACTUATORS/DRAIN_SENSOR_PROBE -> +5V
- R27 pad 2: Net-(Q4-Pad1) -> /AC_ACTUATORS/E3
- R28 pad 1: Net-(Q4-Pad1) -> +5V
- R28 pad 2: GND -> Net-(J8-Pad3)
- R29 pad 1: /DOOR_SENSOR -> /AC_ACTUATORS/E2
- R29 pad 2: GND -> /WATER_LVL_LOW
- R3 pad 1: /DOOR_SENSOR -> +5V
- R3 pad 2: Net-(J4-Pad2) -> Net-(J1-Pad1)
- R30 pad 1: +5V -> /AC_ACTUATORS/E3
- R30 pad 2: /AC_ACTUATORS/E2 -> /WATER_LVL_HIGH
- R31 pad 1: Net-(R31-Pad1) -> Net-(J8-Pad3)
- R31 pad 2: /single_phase_heater_pwm -> /AC_ACTUATORS/DRAIN_SENSOR_PROBE
- R32 pad 1: +5V -> Net-(R32-Pad1)
- R32 pad 2: /AC_ACTUATORS/E3 -> /L2_3phase_heater_pwm
- R33 pad 1: +5V -> Net-(R33-Pad1)
- R33 pad 2: Net-(J8-Pad4) -> /L1_3phase_heater_pwm
- R34 pad 1: L1 -> Net-(R34-Pad1)
- R34 pad 2: Net-(R34-Pad2) -> /L3_3phase_heater_pwm
- R4 pad 2: Net-(D1-Pad2) -> Net-(R4-Pad2)
- R45 pad 1: /AC_ACTUATORS/E2 -> L1
- R45 pad 2: /WATER_LVL_LOW -> Net-(R45-Pad2)
- R5 pad 1: +5V -> Net-(R4-Pad2)
- R5 pad 2: /RESET -> GND
- R6 pad 1: Net-(R6-Pad1) -> +5V
- R6 pad 2: Net-(D2-Pad2) -> Net-(J3-Pad1)
- R7 pad 1: +5V -> /DOOR_SENSOR
- R7 pad 2: /mcu_SCL -> Net-(J4-Pad2)
- R8 pad 1: +5V -> /DOOR_SENSOR
- R8 pad 2: /mcu_SDA -> GND
- R9 pad 1: +3V3 -> +5V
- R9 pad 2: /mcu_SCREEN_RST -> Net-(D1-Pad2)
- RV10 pad 1: Net-(J16-Pad1) -> Net-(J15-Pad1)
- RV11 pad 1: Net-(J15-Pad2) -> Net-(J16-Pad2)
- U1 pad 1: /BIAS -> /TANK_RTD
- U1 pad 2: /BIAS -> Net-(R4-Pad2)
- U1 pad 3: Net-(R1-Pad2) -> Net-(J3-Pad1)
- U1 pad 4: Net-(R1-Pad2) -> GND
- U1 pad 5: Net-(J1-Pad3) -> Net-(J1-Pad1)
- U1 pad 6: Net-(J1-Pad3) -> Net-(R1-Pad2)
- U1 pad 7: /RTD1_IN+ -> /BOILER_RTD
- U1 pad 8: /RTD1_IN- -> +5V
- U2 pad 1: /BIAS1 -> GND
- U2 pad 2: /BIAS1 -> +3V3
- U2 pad 3: Net-(R2-Pad2) -> +5V
- U2 pad 4: Net-(R2-Pad2) -> (no net)
- U3 pad 1: GND -> unconnected-(U3-Pad1)
- U3 pad 2: +3V3 -> /RXD0
- U3 pad 3: +5V -> /TXD0
- U3 pad 4: (no net) -> unconnected-(U3-Pad4)
- U4 pad 1: unconnected-(U4-Pad1) -> Net-(D3-Pad3)
- U4 pad 2: /RXD0 -> GND1
- U4 pad 3: /TXD0 -> /ZERO_CROSS_DETECT
- U4 pad 4: unconnected-(U4-Pad4) -> +5V
- U5 pad 1: Net-(D3-Pad3) -> Net-(R32-Pad1)
- U5 pad 2: GND1 -> GND
- U5 pad 3: /ZERO_CROSS_DETECT -> unconnected-(U5-Pad3)
- U5 pad 4: +5V -> Net-(D7-Pad3)
- U6 pad 1: Net-(R21-Pad1) -> Net-(R33-Pad1)
- U6 pad 4: Net-(D4-Pad3) -> Net-(D8-Pad3)
- U6 pad 6: Net-(R24-Pad2) -> Net-(R36-Pad2)
- U7 pad 1: Net-(R22-Pad1) -> Net-(R34-Pad1)
- U7 pad 4: Net-(D5-Pad3) -> Net-(D9-Pad3)
- U7 pad 6: Net-(R25-Pad2) -> Net-(R37-Pad2)
- U8 pad 1: Net-(R23-Pad1) -> Net-(R44-Pad1)
- U8 pad 4: Net-(D6-Pad3) -> Net-(D13-Pad3)
- U8 pad 6: Net-(R26-Pad2) -> Net-(R45-Pad2)
- Y1 pad 1: Net-(C14-Pad1) -> Net-(C8-Pad1)
- Y1 pad 3: Net-(C15-Pad1) -> Net-(C9-Pad1)
Routing:
- net +5V: track 491.4 -> 583.3 mm, vias 14 -> 11
- net +3V3: track 122.5 -> 39.8 mm, vias 10 -> 2
- net /RTD_SCLK: track 81.9 -> 0.00 mm, vias 4 -> 0
- net /MOSI: track 86.4 -> 37.4 mm
- net GND: track 210.0 -> 256.5 mm, vias 55 -> 51
- net /SCK: track 0.00 -> 42.9 mm, vias 0 -> 2
- net /peristaltic_pump_1: track 84.8 -> 43.9 mm, vias 4 -> 2
- net /L3_3phase_heater_pwm: track 39.7 -> 76.4 mm
- net /RTD_~{DRDY_1}: track 36.5 -> 0.00 mm, vias 4 -> 0
- net /MISO: track 70.5 -> 38.0 mm, vias 4 -> 2
- net /BOILER_RTD: track 0.00 -> 30.3 mm, vias 0 -> 2
- net /TANK_RTD: track 0.00 -> 28.4 mm, vias 0 -> 2
- net /peristaltic_pump_2: track 68.0 -> 95.5 mm
- net /RTD1_IN-: track 26.7 -> 0.00 mm
- net /RTD1_IN+: track 22.9 -> 0.00 mm
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- added copper zone on In1.Cu, net L3
- added copper zone on In1.Cu, net NEUTRAL
- added copper zone on In1.Cu, net Net-(J15-Pad1)
- added copper zone on In1.Cu, net Net-(J16-Pad2)
- removed copper zone on F.Cu, net Net-(J15-Pad2)
- removed copper zone on B.Cu, net Net-(J16-Pad1)
Other:
- board text added: "MISO"
- board text added: "MOSI"
- board text added: "RST"
- board text added: "SCK"
- board text removed: "X"

Commit message: layput update
Parts:
- moved R43 3.14 mm to (163.2, 73.0), turned to 90 degrees
- moved C9 2.19 mm to (231.7, 124.7)
- moved C8 1.84 mm to (231.6, 130.0)
- moved Y1 1.82 mm to (231.7, 127.3)
- moved J2 1.80 mm to (135.2, 89.7)
- moved J15 1.71 mm to (249.3, 64.2)
- moved J16 1.71 mm to (169.1, 64.2)
- moved J17 1.60 mm to (287.1, 69.8)
- moved J12 1.40 mm to (212.2, 69.9)
- moved SW1 0.15 mm to (237.3, 117.2)
- moved J14 0.12 mm to (218.5, 145.5)
Routing:
- net GND: track 256.5 -> 221.5 mm, vias 51 -> 49
- net /L1_3phase_heater_pwm: track 92.4 -> 106.1 mm, vias 2 -> 4
- net /peristaltic_pump_2: track 95.5 -> 106.1 mm
- net /peristaltic_pump_1: track 43.9 -> 52.4 mm
- net +5V: track 583.3 -> 590.8 mm, vias 11 -> 15
- net /SPEAKER: track 55.6 -> 63.0 mm
- net /single_phase_heater_pwm: track 96.7 -> 102.6 mm
- net /L3_3phase_heater_pwm: track 76.4 -> 82.0 mm
- net /ZERO_CROSS_DETECT: track 68.2 -> 73.5 mm
- net Net-(Q6-Pad1): track 8.52 -> 3.28 mm
- net /RESET: track 44.0 -> 49.2 mm
- net /MOSI: track 37.4 -> 42.3 mm
- net /mcu_~{IRQ}: track 56.7 -> 61.2 mm
- net /mcu_SDA: track 56.8 -> 61.1 mm
- net /mcu_SCL: track 57.6 -> 61.6 mm
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Other:
- board text added: "DET"
- board text added: "Drain"
- board text added: "ELEMENT1"
- board text added: "ELEMENT2"
- board text added: "ELEMENT3"
- board text added: "HEATER"
- board text added: "L"
- board text added: "L1"
- board text added: "L2"
- board text added: "L3"
- board text added: "N"
- board text added: "NEUTRAL"
- board text added: "RESET"
- board text added: "RINSE"
- board text added: "SOLENOID"
- board text added: "Wash"
