File: dish_washwer_hardware/src/Steel_form_Dish_washer PART 2.kicad_pcb (KiCad board)
At the start: 4 copper layers, 230 x 35 mm, 25 parts, among them J18 Conn_02x07_Odd_Even, J19 SCREEN CONNECTOR, J20 Conn_01x10_Male, U12 TXS0108EPW, U13 EAST1616RGBA8, U14 EAST1616RGBA8, U15 MPR121QR2

Commit message: complete layout and schematic
Parts:
- removed C23, C24: 100nF, Capacitor_SMD:C_0402_1005Metric
- removed R35, R37, R38, R40: 100R, Resistor_SMD:R_0603_1608Metric
- removed R36, R39: 150R, Resistor_SMD:R_0603_1608Metric
- removed R41, R42, R44: 4.7K, Resistor_SMD:R_0603_1608Metric
- removed R43: 75K, Resistor_SMD:R_0603_1608Metric
- removed U13, U14: EAST1616RGBA8, greencharge-footprints:EAST1616RGBA8
- removed U15: MPR121QR2, Package_DFN_QFN:UQFN-20_3x3mm_P0.4mm
- added C17: 100nF, Capacitor_SMD:C_0402_1005Metric, F.Cu at (192.0, 229.2)
- added C18: 100nF, Capacitor_SMD:C_0402_1005Metric, F.Cu at (193.1, 221.9)
- added R46: 100R, Resistor_SMD:R_0603_1608Metric, F.Cu at (92.2, 236.7)
- added R47: 150R, Resistor_SMD:R_0603_1608Metric, F.Cu at (94.0, 236.7)
- added R48: 100R, Resistor_SMD:R_0603_1608Metric, F.Cu at (95.9, 236.7)
- added R49: 100R, Resistor_SMD:R_0603_1608Metric, F.Cu at (280.9, 236.2)
- added R50: 150R, Resistor_SMD:R_0603_1608Metric, F.Cu at (282.8, 236.2)
- added R51: 100R, Resistor_SMD:R_0603_1608Metric, F.Cu at (284.4, 236.2)
- added R53: 4.7K, Resistor_SMD:R_0603_1608Metric, F.Cu at (296.1, 236.4)
- added R54: 75K, Resistor_SMD:R_0603_1608Metric, F.Cu at (193.4, 229.7)
- added R55: 4.7K, Resistor_SMD:R_0603_1608Metric, F.Cu at (296.1, 238.1)
- added R56: 4.7K, Resistor_SMD:R_0402_1005Metric, F.Cu at (279.5, 235.5)
- added U10: EAST1616RGBA8, greencharge-footprints:EAST1616RGBA8, F.Cu at (93.3, 240.6)
- added U11: EAST1616RGBA8, greencharge-footprints:EAST1616RGBA8, F.Cu at (281.8, 241.0)
- added U9: TXS0108EPW, Package_SO:TSSOP-20_4.4x6.5mm_P0.65mm, B.Cu at (289.1, 237.8)
- R52: footprint Resistor_SMD:R_0402_1005Metric -> Resistor_SMD:R_0603_1608Metric
- U12: value TXS0108EPW -> MPR121QR2; footprint Package_SO:TSSOP-20_4.4x6.5mm_P0.65mm -> Package_DFN_QFN:UQFN-20_3x3mm_P0.4mm; moved to F.Cu
- moved U12 90.4 mm to (194.0, 225.1), turned to 0 degrees
- moved R52 16.6 mm to (296.1, 234.8), turned to 180 degrees
Connections:
- R52 pad 2: /PCB 2/SCREEN_RST -> /PCB 2/SDA
- U12 pad 1: /PCB 2/SDA -> /PCB 2/~{IRQ}
- U12 pad 10: +3V3 -> /PCB 2/BACK
- U12 pad 11: GND -> /PCB 2/LEFT
- U12 pad 12: unconnected-(U12-Pad12) -> /PCB 2/SET
- U12 pad 13: unconnected-(U12-Pad13) -> /PCB 2/RIGHT
- U12 pad 14: unconnected-(U12-Pad14) -> /PCB 2/START
- U12 pad 16: /PCB 2/mcu_SCREEN_RST -> unconnected-(U12-Pad16)
- U12 pad 17: /PCB 2/mcu_~{IRQ} -> unconnected-(U12-Pad17)
- U12 pad 18: /PCB 2/mcu_SCL -> unconnected-(U12-Pad18)
- U12 pad 19: +5V -> unconnected-(U12-Pad19)
- U12 pad 2: +3V3 -> /PCB 2/SCL
- U12 pad 20: /PCB 2/mcu_SDA -> +3V3
- U12 pad 3: /PCB 2/SCL -> /PCB 2/SDA
- U12 pad 4: /PCB 2/~{IRQ} -> GND
- U12 pad 5: /PCB 2/SCREEN_RST -> Net-(C17-Pad1)
- U12 pad 6: unconnected-(U12-Pad6) -> GND
- U12 pad 7: unconnected-(U12-Pad7) -> Net-(R54-Pad1)
- U12 pad 8: unconnected-(U12-Pad8) -> /PCB 2/ON/OFF
- U12 pad 9: unconnected-(U12-Pad9) -> /PCB 2/MENU
Routing:
- net /PCB 2/SDA: track 185.6 -> 134.4 mm, vias 0 -> 4
- net /PCB 2/RGB_ON/OFF_BLU: track 239.5 -> 203.6 mm, vias 5 -> 2
- net /PCB 2/SCL: track 171.7 -> 137.5 mm, vias 0 -> 4
- net /PCB 2/START: track 67.1 -> 35.0 mm
- net /PCB 2/RGB_ON/OFF_RED: track 236.1 -> 205.6 mm, vias 5 -> 3
- net /PCB 2/RIGHT: track 63.8 -> 36.3 mm
- net /PCB 2/RGB_ON/OFF_GRN: track 225.0 -> 203.6 mm, vias 3 -> 2
- net +3V3: track 163.7 -> 173.1 mm, vias 6 -> 4
- net GND: track 12.3 -> 3.09 mm, vias 26 -> 24
- net /PCB 2/~{IRQ}: track 120.9 -> 129.7 mm, vias 1 -> 4
- net /PCB 2/mcu_SDA: track 7.92 -> 15.9 mm
- net +5V: track 9.40 -> 16.6 mm
- net /PCB 2/mcu_SCL: track 7.53 -> 14.1 mm
- net /PCB 2/SCREEN_RST: track 18.0 -> 24.0 mm
- net /PCB 2/mcu_~{IRQ}: track 20.2 -> 24.4 mm
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